File: 3D robot.kicad_sch (KiCad schematic)
At the start: 29 parts

Commit message: reference designator added
Parts:
- gave numbers to parts that had none: 29

Commit message: updating schematics
Parts:
- removed A1, A2, A3: Arduino_Nano_v3.x, Module:Arduino_Nano, symbol MCU_Module:Arduino_Nano_v3.x
- removed BT1: Battery_Cell, symbol Device:Battery_Cell
- removed D1, D2: RB161QS-40, my_footprints:RB161QS-40T18R, symbol diodes:RB161QS-40
- removed J1: Raspberry_Pi_2_3, symbol Connector:Raspberry_Pi_2_3
- removed M1, M18: Motor_DC, symbol Motor:Motor_DC
- removed M10, M11, M15, M16, M19, M20, M3, M7, M8, M9: Stepper_Motor_bipolar, symbol Motor:Stepper_Motor_bipolar
- removed M12, M13, M14, M4, M5, M6: Motor_Servo, symbol Motor:Motor_Servo
- removed M17, M2: RHP020N06, my_footprints:RHP020N06T100, symbol E-MOSFETs:RHP020N06
- removed R1, R2: 11, my_footprints:MCR03EZPFX, symbol resistors:MCR03EZPFX
Other:
- removed sheet Buck converter 5 and 12
- removed sheet Buck converter 7.4
- removed sheet stepper and controller
- removed sheet stepper and controller1
- removed sheet stepper and controller2
- removed sheet stepper and controller3
- removed sheet stepper and controller4
- removed sheet stepper and controller5
- removed sheet stepper and controller6
- removed sheet stepper and controller7
- removed sheet stepper and controller8
- removed sheet stepper and controller9
- added sheet Base (base.kicad_sch)
- added sheet Left arm (left arm.kicad_sch)
- added sheet Right arm (right arm.kicad_sch)
