File: base TH.kicad_pcb (KiCad board)
At the start: 2 copper layers, 156.5 x 113.8 mm, 35 parts, among them J1 282856-8, J2 Raspberry_Pi_2_3, M1 Stepper_Motor_bipolar, M2 Stepper_Motor_bipolar, M3 Stepper_Motor_bipolar, M4 Stepper_Motor_bipolar, U1 TMC2209 silent step stick, U2 TMC2209 silent step stick, U3 TMC2209 silent step stick, U4 TMC2209 silent step stick

Commit message: stitching updated
Parts:
- added U5: LM2596, base TH:LM2596, F.Cu at (226.5, 140.4)
Routing:
- net /-: vias 266 -> 249
- added copper zone on F.Cu, net /-
